File: washington-metro-pcb_single_stations/washington-metro-pcb.kicad_sch (KiCad schematic)
At the start: 202 parts, among them J1 Conn_01x04, U1 74AHC1G125

Commit message: As sent to JLCPCB 2024-March-23
Parts:
- J1: value Conn_01x04 -> Conn_01x05; footprint Connector_PinHeader_2.54mm:PinHeader_1x04_P2.54mm_Vertical -> Connector_PinHeader_2.54mm:PinHeader_1x05_P2.54mm_Vertical; symbol Connector_Generic:Conn_01x04 -> Connector_Generic:Conn_01x05
Connections:
- net LED_ROW_ONE_IN: now also J1.5 (Pin_5)
